Commit message: update: Kinect scan converted to stanalone, Depth to laser implemented to main launch

File: description/robot.urdf.xacro (robot description, xacro)
@@ -2,4 +2,6 @@
 <robot xmlns:xacro="http://www.ros.org/wiki/xacro" name="robot">
     <xacro:arg name="use_ros2_control" default="true"/>
+    <!-- //////////////////////////////////////////////////////////////////////////////////////// -->
+    <!-- ////////////////////////Constants////////////////////////////////////////////////////// -->
     <!-- Macros for Inertials -->
     <xacro:macro name="inertial_sphere" params="mass radius *origin">
@@ -30,4 +32,6 @@
         </inertial>
     </xacro:macro>
+    <!-- //////////////////////////////////////////////////////////////////////////////////////// -->
+    <!-- ////////////////////////Constants////////////////////////////////////////////////////// -->
     <!-- Materials -->
     <material name="white">
@@ -46,4 +50,6 @@
         <color rgba="1 0.3 0.1 1" />
     </material>
+    <!-- //////////////////////////////////////////////////////////////////////////////////////// -->
+    <!-- ////////////////////////Base/////////////////////////////////////////////////////////// -->
     <!-- Base Link -->
     <link name="base_link"/>
@@ -55,4 +61,6 @@
     </joint>
     <link name="base_footprint"/>
+    <!-- //////////////////////////////////////////////////////////////////////////////////////// -->
+    <!-- ////////////////////////Chassis//////////////////////////////////////////////////////// -->
     <!-- Chassis Link -->
     <joint name="chassis_joint" type="fixed">
@@ -147,4 +155,6 @@
         <material>Gazebo/White</material>
     </gazebo>
+    <!-- //////////////////////////////////////////////////////////////////////////////////////// -->
+    <!-- ////////////////////////Wheels///////////////////////////////////////////////////////// -->
     <!-- Left Wheel Link -->
     <joint name="left_wheel_joint" type="continuous">
@@ -227,4 +237,6 @@
         <mu2 value="0.001"/>
     </gazebo>
+    <!-- //////////////////////////////////////////////////////////////////////////////////////// -->
+    <!-- ////////////////////////Gazebo Plugins///////////////////////////////////////////////// -->
     <!-- Control Selection -->
     <xacro:if value="$(arg use_ros2_control)">
@@ -276,17 +288,13 @@
         </gazebo>
     </xacro:unless>
-    <!-- Laser Joint and Link -->
-    <joint name="laser_joint" type="fixed">
+    <!-- //////////////////////////////////////////////////////////////////////////////////////// -->
+    <!-- ////////////////////////Counter Weight///////////////////////////////////////////////// -->
+    <!-- counter weight -->
+    <joint name="counter_weight_joint" type="fixed">
         <parent link="chassis"/>
-        <child link="laser_frame"/>
+        <child link="counter_weight_frame"/>
         <origin xyz="0.1 0 0.13" rpy="0 0 0"/>
     </joint>
-    <link name="laser_frame">
-        <visual>
-            <geometry>
-                <cylinder radius="0.05" length="0.04"/>
-            </geometry>
-            <material name="red"/>
-        </visual>
+    <link name="counter_weight_frame">
         <collision>
             <geometry>
@@ -298,183 +306,66 @@
         </xacro:inertial_cylinder>
     </link>
-<!--
+    <!-- //////////////////////////////////////////////////////////////////////////////////////// -->
+    <!-- ////////////////////////Kinect V2/////////////////////////////////////////////////////// -->
+    <!-- Kinect Link -->
+    <link name="laser_frame">
+        <visual>
+        <geometry>
+            <box size="0.05 0.23 0.04"/>
+        </geometry>
+        <origin xyz="0.13 0 0.26" rpy="0 0 0"/>
+        <material name="black"/>
+        </visual>
+    </link>
+    <!-- Kinect Joint -->
+    <joint name="laser_joint" type="fixed">
+        <parent link="base_link"/>
+        <child link="laser_frame"/>
+        <origin xyz="0 0 0.5" rpy="0 0 0"/>
+    </joint>
+    <!-- Kinect Gazebo Configuration -->
     <gazebo reference="laser_frame">
         <material>Gazebo/Black</material>
-        <sensor type="ray" name="laser">
-            <pose>0 0 0 0 0 0</pose>
-            <visualize>false</visualize>
-            <update_rate>10</update_rate>
-            <ray>
-                <scan>
-                    <horizontal>
-                        <samples>360</samples>
-                        <resolution>1</resolution>
-                        <min_angle>-3.14</min_angle>
-                        <max_angle>3.14</max_angle>
-                    </horizontal>
-                </scan>
-                <range>
-                    <min>0.3</min>
-                    <max>12</max>
-                    <resolution>0.01</resolution>
-                </range>
-            </ray>
-            <plugin name="laser_controller" filename="libgazebo_ros_ray_sensor.so">
-                <ros>
-                    <argument>~/out:=scan</argument>
-                </ros>
-                <output_type>sensor_msgs/LaserScan</output_type>
-                <frameName>laser_frame</frameName>
-            </plugin>
+        <sensor type="depth" name="kinect_depth">
+        <update_rate>30</update_rate>
+        <pose>0 0 0 0 0 0</pose>
+        <visualize>true</visualize>
+        <depth>
+            <clip>
+            <near>0.1</near>
+            <far>10.0</far>
+            </clip>
+            <horizontal_fov>1.047</horizontal_fov>
+        </depth>
+        <camera>
+            <horizontal_fov>1.047</horizontal_fov>
+            <image>
+            <width>640</width>
+            <height>480</height>
+            <format>R8G8B8</format>
+            </image>
+            <clip>
+            <near>0.1</near>
+            <far>10.0</far>
+            </clip>
+        </camera>
+        <plugin name="kinect_camera_controller" filename="libgazebo_ros_camera.so">
+            <alwaysOn>true</alwaysOn>
+            <updateRate>0.0</updateRate>
+            <cameraName>kinect_rgb</cameraName>
+        </plugin>
+        <plugin name="depth_camera_controller" filename="libgazebo_ros_depth_camera.so">
+            <alwaysOn>true</alwaysOn>
+            <updateRate>0.0</updateRate>
+            <cameraName>kinect_depth</cameraName>
+        </plugin>
         </sensor>
-    </gazebo> -->
-    <!-- Camera Joint and Link -->
-    <!-- <joint name="camera_joint" type="fixed">
-        <parent link="chassis"/>
-        <child link="camera_link"/>
-        <origin xyz="0.305 0 0.12" rpy="0 0 0"/>
-    </joint>
-    <link name="camera_link">
-        <visual>
-            <geometry>
-                <box size="0.010 0.03 0.03"/>
-            </geometry>
-            <material name="red"/>
-        </visual>
-    </link>
-    <joint name="camera__optical_joint" type="fixed">
-        <parent link="camera_link"/>
-        <child link="camera_link_optical"/>
-        <origin xyz="0 0 0" rpy="${-pi/2} 0 ${-pi/2}"/>
-    </joint>
-    <link name="camera_link_optical"/>
-    <gazebo reference="camera_link">
-        <material>Gazebo/Black</material>
-        <sensor type="camera" name="camera">
-            <pose>0 0 0 0 0 0</pose>
-            <visualize>false</visualize>
-            <update_rate>10</update_rate>
-            <camera>
-                <horizontal_fov>1.089</horizontal_fov>
-                <image>
-                    <width>640</width>
-                    <height>480</height>
-                    <format>R8G8B8</format>
-                </image>
-                <clip>
-                    <near>0.05</near>
-                    <far>8.0</far>
-                </clip>
-            </camera>
-            <plugin name="camera_controller" filename="libgazebo_ros_camera.so">
-                <frameName>camera_link_optical</frameName>
-            </plugin>
-        </sensor>
-    </gazebo> -->
-<!--
-      <joint name="camera_joint" type="fixed">
-        <parent link="chassis"/>
-        <child link="camera_link"/>
-        <origin xyz="0.305 0 0.08" rpy="0 0 0"/>
-    </joint>
-    <link name="camera_link">
-        <visual>
-            <geometry>
-                <box size="0.010 0.03 0.03"/>
-            </geometry>
-            <material name="red"/>
-        </visual>
-    </link>
-    <joint name="camera_optical_joint" type="fixed">
-        <parent link="camera_link"/>
-        <child link="camera_link_optical"/>
-        <origin xyz="0 0 0" rpy="${-pi/2} 0 ${-pi/2}"/>
-    </joint>
-    <link name="camera_link_optical"></link>
-    <gazebo reference="camera_link">
-        <material>Gazebo/Red</material>
-        <sensor name="camera" type="depth">
-            <pose> 0 0 0 0 0 0 </pose>
-            <visualize>true</visualize>
-            <update_rate>10</update_rate>
-            <camera>
-                <horizontal_fov>1.089</horizontal_fov>
-                <image>
-                    <format>B8G8R8</format>
-                    <width>640</width>
-                    <height>480</height>
-                </image>
-                <clip>
-                    <near>0.05</near>
-                    <far>8.0</far>
-                </clip>
-            </camera>
-            <plugin name="camera_controller" filename="libgazebo_ros_camera.so">
-                <frame_name>camera_link_optical</frame_name>
-                <min_depth>0.1</min_depth>
-                <max_depth>100.0</max_depth>
-            </plugin>
-        </sensor>
-    </gazebo> -->
-    <!-- Kinect Link -->
-  <link name="kinect_link">
-    <visual>
-      <geometry>
-        <box size="0.05 0.23 0.04"/>
-      </geometry>
-      <origin xyz="0.13 0 0.26" rpy="0 0 0"/>
-      <material name="black"/>
-    </visual>
-  </link>
-  <!-- Kinect Joint -->
-  <joint name="kinect_joint" type="fixed">
-    <parent link="base_link"/>
-    <child link="kinect_link"/>
-    <origin xyz="0 0 0.5" rpy="0 0 0"/>
-  </joint>
-  <!-- Kinect Gazebo Configuration -->
-  <gazebo reference="kinect_link">
-    <material>Gazebo/Black</material>
-    <sensor type="depth" name="kinect_depth">
-      <update_rate>30</update_rate>
-      <pose>0 0 0 0 0 0</pose>
-      <visualize>true</visualize>
-      <depth>
-        <clip>
-          <near>0.1</near>
-          <far>10.0</far>
-        </clip>
-        <horizontal_fov>1.047</horizontal_fov>
-      </depth>
-      <camera>
-        <horizontal_fov>1.047</horizontal_fov>
-        <image>
-          <width>640</width>
-          <height>480</height>
-          <format>R8G8B8</format>
-        </image>
-        <clip>
-          <near>0.1</near>
-          <far>10.0</far>
-        </clip>
-      </camera>
-      <plugin name="kinect_camera_controller" filename="libgazebo_ros_camera.so">
+    </gazebo>
+    <gazebo>
+        <plugin name="gazebo_ros_openni_kinect" filename="libgazebo_ros_openni_kinect.so">
         <alwaysOn>true</alwaysOn>
         <updateRate>0.0</updateRate>
-        <cameraName>kinect_rgb</cameraName>
-      </plugin>
-      <plugin name="depth_camera_controller" filename="libgazebo_ros_depth_camera.so">
-        <alwaysOn>true</alwaysOn>
-        <updateRate>0.0</updateRate>
-        <cameraName>kinect_depth</cameraName>
-      </plugin>
-    </sensor>
-  </gazebo>
-  <gazebo>
-    <plugin name="gazebo_ros_openni_kinect" filename="libgazebo_ros_openni_kinect.so">
-      <alwaysOn>true</alwaysOn>
-      <updateRate>0.0</updateRate>
-      <cameraName>kinect</cameraName>
-    </plugin>
-  </gazebo>
+        <cameraName>kinect</cameraName>
+        </plugin>
+    </gazebo>
 </robot>

Commit message: update: Actuators done with ros2_control

File: description/robot.urdf.xacro (robot description, xacro)
@@ -142,4 +142,12 @@
             <material name="orange"/>
         </visual>
+        <visual>
+            <!-- Third Deck -->
+            <origin xyz="0.15 0 0.5"/> <!-- Adjusted for height of first deck plus poles -->
+            <geometry>
+                <box size="0.3 0.3 0.1"/>
+            </geometry>
+            <material name="orange"/>
+        </visual>
         <collision>
             <origin xyz="0.15 0 0.075"/>
@@ -240,52 +248,62 @@
     <!-- ////////////////////////Gazebo Plugins///////////////////////////////////////////////// -->
     <!-- Control Selection -->
-    <xacro:if value="$(arg use_ros2_control)">
-        <ros2_control name="GazeboSystem" type="system">
-            <hardware>
-                <plugin>gazebo_ros2_control/GazeboSystem</plugin>
-            </hardware>
-            <joint name="left_wheel_joint">
-                <command_interface name="velocity">
-                    <param name="min"></param>
-                    <param name="max"></param>
-                </command_interface>
-                <state_interface name="velocity"/>
-                <state_interface name="position"/>
-            </joint>
-            <joint name="right_wheel_joint">
-                <command_interface name="velocity">
-                    <param name="min"></param>
-                    <param name="max"></param>
-                </command_interface>
-                <state_interface name="velocity"/>
-                <state_interface name="position"/>
-            </joint>
-        </ros2_control>
-        <gazebo>
-            <plugin name="gazebo_ros2_control" filename="libgazebo_ros2_control.so">
-                <parameters>$(find SLAM_ros2_bot)/config/my_parameters.yaml</parameters>
-            </plugin>
-        </gazebo>
-    </xacro:if>
-    <xacro:unless value="$(arg use_ros2_control)">
-        <gazebo>
-            <plugin name="diff_drive" filename="libgazebo_ros_diff_drive.so">
-                <!-- wheel information -->
-                <left_joint>left_wheel_joint</left_joint>
-                <right_joint>right_wheel_joint</right_joint>
-                <wheel_separation>0.35</wheel_separation>
-                <wheel_diameter>0.1</wheel_diameter>
-                <!-- limits -->
-                <max_wheel_torque>200</max_wheel_torque>
-                <max_wheel_acceleration>10.0</max_wheel_acceleration>
-                <!-- Outputs -->
-                <odometry_frame>odom</odometry_frame>
-                <robot_base_frame>base_link</robot_base_frame>
-                <publish_odom>true</publish_odom>
-                <publish_odom_tf>true</publish_odom_tf>
-                <publish_wheel_tf>true</publish_wheel_tf>
-            </plugin>
-        </gazebo>
-    </xacro:unless>
+    <ros2_control name="GazeboSystem" type="system">
+        <hardware>
+            <plugin>gazebo_ros2_control/GazeboSystem</plugin>
+        </hardware>
+        <joint name="left_wheel_joint">
+            <command_interface name="velocity">
+                <param name="min"></param>
+                <param name="max"></param>
+            </command_interface>
+            <state_interface name="velocity"/>
+            <state_interface name="position"/>
+        </joint>
+        <joint name="right_wheel_joint">
+            <command_interface name="velocity">
+                <param name="min"></param>
+                <param name="max"></param>
+            </command_interface>
+            <state_interface name="velocity"/>
+            <state_interface name="position"/>
+        </joint>
+        <joint name="left_arm_joint">
+            <command_interface name="position">
+                <param name="min"></param>
+                <param name="max"></param>
+            </command_interface>
+            <state_interface name="velocity"/>
+            <state_interface name="position"/>
+        </joint>
+        <joint name="right_arm_2_joint">
+            <command_interface name="position">
+                <param name="min"></param>
+                <param name="max"></param>
+            </command_interface>
+            <state_interface name="velocity"/>
+            <state_interface name="position"/>
+        </joint>
+        <joint name="left_arm_2_joint">
+            <command_interface name="position">
+                <param name="min"></param>
+                <param name="max"></param>
+            </command_interface>
+            <state_interface name="velocity"/>
+            <state_interface name="position"/>
+        </joint>
+        <joint name="right_arm_joint">
+            <command_interface name="position">
+                <param name="min"></param>
+                <param name="max"></param>
+            </command_interface>
+            <state_interface name="velocity"/>
+            <state_interface name="position"/>
+        </joint>
+    </ros2_control>
+    <gazebo>
+        <plugin name="gazebo_ros2_control" filename="libgazebo_ros2_control.so">
+            <parameters>$(find SLAM_ros2_bot)/config/my_parameters.yaml</parameters>
+        </plugin>
+    </gazebo>
     <!-- //////////////////////////////////////////////////////////////////////////////////////// -->
     <!-- ////////////////////////Counter Weight///////////////////////////////////////////////// -->
@@ -306,4 +324,133 @@
         </xacro:inertial_cylinder>
     </link>
+    <!-- //////////////////////////////////////////////////////////////////////////////////////// -->
+    <!-- ////////////////////////Left arm/////////////////////////////////////////////////////// -->
+    <!-- Left Arm Link -->
+    <joint name="left_arm_joint" type="continuous">
+        <parent link="base_link"/>
+        <child link="left_arm_1"/>
+        <origin xyz="0 0.175 0.5" rpy="-${pi/2} 0 0.2"/>
+        <axis xyz="0 0 1"/>
+    </joint>
+    <link name="left_arm_1">
+        <visual>
+            <geometry>
+                <box size="0.4 0.05 0.05"/>
+            </geometry>
+            <origin xyz="0.175 0 0.005"/>
+            <material name="white"/>
+        </visual>
+        <collision>
+            <geometry>
+                <box size="0.4 0.05 0.05"/>
+            </geometry>
+            <origin xyz="0.175 0 0.005"/>
+        </collision>
+        <xacro:inertial_cylinder mass="0.0001" length="0.04" radius="0.05">
+            <origin xyz="0 0 0" rpy="0 0 0"/>
+        </xacro:inertial_cylinder>
+    </link>
+    <joint name="left_arm_2_joint" type="continuous">
+        <parent link="left_arm_1"/>
+        <child link="left_arm_2"/>
+        <origin xyz="0.36 -0.05 0" rpy="0 0 0"/>
+        <axis xyz="0 1 0"/>
+    </joint>
+    <link name="left_arm_2">
+        <visual>
+            <geometry>
+                <box size="0.3 0.05 0.05"/>
+            </geometry>
+            <origin xyz="0.14 0 0.005"/>
+            <material name="white"/>
+        </visual>
+        <collision>
+            <geometry>
+                <sphere radius="0.05"/>
+            </geometry>
+        </collision>
+        <xacro:inertial_cylinder mass="0.0001" length="0.04" radius="0.05">
+            <origin xyz="0 0 0" rpy="0 0 0"/>
+        </xacro:inertial_cylinder>
+    </link>
+    <gazebo reference="left_arm_1">
+        <material>Gazebo/White</material>
+    </gazebo>
+    <gazebo reference="left_arm_2">
+        <material>Gazebo/White</material>
+    </gazebo>
+    <!-- //////////////////////////////////////////////////////////////////////////////////////// -->
+    <!-- ////////////////////////Right arm////////////////////////////////////////////////////// -->
+    <!-- Right Arm Link -->
+    <joint name="right_arm_joint" type="continuous">
+        <parent link="base_link"/>
+        <child link="right_arm_1"/>
+        <origin xyz="0 -0.175 0.5" rpy="${pi/2} 0 -0.2"/>
+        <axis xyz="0 0 -1"/>
+    </joint>
+    <link name="right_arm_1">
+        <visual>
+            <geometry>
+                <box size="0.4 0.05 0.05"/>
+            </geometry>
+            <origin xyz="0.175 0 0.005"/>
+            <material name="white"/>
+        </visual>
+        <collision>
+            <geometry>
+                <sphere radius="0.05"/>
+            </geometry>
+        </collision>
+        <xacro:inertial_cylinder mass="0.0001" length="0.04" radius="0.05">
+            <origin xyz="0 0 0" rpy="0 0 0"/>
+        </xacro:inertial_cylinder>
+    </link>
+    <joint name="right_arm_2_joint" type="continuous">
+        <parent link="right_arm_1"/>
+        <child link="right_arm_2"/>
+        <origin xyz="0.36 0.05 0" rpy="0 0 0"/>
+        <axis xyz="0 1 0"/>
+    </joint>
+    <link name="right_arm_2">
+        <visual>
+            <geometry>
+                <box size="0.3 0.05 0.05"/>
+            </geometry>
+            <origin xyz="0.14 0 0.005"/>
+            <material name="white"/>
+        </visual>
+        <collision>
+            <geometry>
+                <sphere radius="0.05"/>
+            </geometry>
+        </collision>
+        <xacro:inertial_cylinder mass="0.0001" length="0.04" radius="0.05">
+            <origin xyz="0 0 0" rpy="0 0 0"/>
+        </xacro:inertial_cylinder>
+    </link>
+    <gazebo reference="right_arm_1">
+        <material>Gazebo/White</material>
+    </gazebo>
+    <gazebo reference="right_arm_2">
+        <material>Gazebo/White</material>
+    </gazebo>
+    <!-- //////////////////////////////////////////////////////////////////////////////////////// -->
+    <!-- ////////////////////////Ros control for arms/////////////////////////////////////////////////////// -->
+    <!-- <gazebo>
+        <plugin name="gazebo_ros_control" filename="libgazebo_ros_control.so">
+            <robotNamespace>/arm_control</robotNamespace>
+            <robotSimType>gazebo_ros_control/DefaultRobotHWSim</robotSimType>
+        </plugin>
+    </gazebo>
+     <transmission name="left_joint_1">
+        <type>transmission_interface/SimpleTransmission</type>
+        <joint name="left_arm_joint">
+        <hardwareInterface>EffortJointInterface</hardwareInterface>
+        </joint>
+        <actuator name="right_arm_1">
+        <hardwareInterface>EffortJointInterface</hardwareInterface>
+        <mechanicalReduction>1</mechanicalReduction>
+        </actuator>
+    </transmission> -->
     <!-- //////////////////////////////////////////////////////////////////////////////////////// -->
     <!-- ////////////////////////Kinect V2/////////////////////////////////////////////////////// -->
